File: PCBs/Remote/CenterBoard/Power.sch (KiCad schematic (older format))
At the start: 4 parts, among them U401 SC189ZSKTRT

Commit message: Bezig met LEDS
Signed-off-by: Eldalote.Electronics <Eldalote.Electronics@gmail.com>
Parts:
- renumbered C401 to C301, C404 to C302, L401 to L301, U401 to U301
Changed lines of the file:
@@
 $Descr A4 11693 8268
 encoding utf-8
-Sheet 3 4
+Sheet 3 5
 Title ""
 Date ""
@@
 $EndDescr
 $Comp
-L SamacSys_Parts:SC189ZSKTRT U401
+L SamacSys_Parts:SC189ZSKTRT U301
 U 1 1 5F640727
 P 5150 2900
-F 0 "U401" H 5625 3165 50  0000 C CNN
+F 0 "U301" H 5625 3165 50  0000 C CNN
 F 1 "SC189ZSKTRT" H 5625 3074 50  0000 C CNN
 F 2 "SOT95P280X145-5N" H 6100 3000 50  0001 L CNN
@@
 $EndComp
 $Comp
-L Device:C_Small C404
+L Device:C_Small C302
 U 1 1 5F641444
 P 6800 3050
-F 0 "C404" H 6892 3096 50  0000 L CNN
+F 0 "C302" H 6892 3096 50  0000 L CNN
 F 1 "22uF" H 6892 3005 50  0000 L CNN
 F 2 "Capacitor_SMD:C_0805_2012Metric_Pad1.15x1.40mm_HandSolder" H 6800 3050 50  0001 C CNN
@@
 $EndComp
 $Comp
-L Device:C_Small C401
+L Device:C_Small C301
 U 1 1 5F64184D
 P 4500 3050
-F 0 "C401" H 4592 3096 50  0000 L CNN
+F 0 "C301" H 4592 3096 50  0000 L CNN
 F 1 "10uF" H 4592 3005 50  0000 L CNN
 F 2 "Capacitor_SMD:C_0805_2012Metric_Pad1.15x1.40mm_HandSolder" H 4500 3050 50  0001 C CNN
@@
 $EndComp
 $Comp
-L Device:L L401
+L Device:L L301
 U 1 1 5F641EA5
 P 6450 2900
-F 0 "L401" V 6640 2900 50  0000 C CNN
+F 0 "L301" V 6640 2900 50  0000 C CNN
 F 1 "1uH" V 6549 2900 50  0000 C CNN
 F 2 "Eldalote-footprints:L_3012_TDK" H 6450 2900 50  0001 C CNN
@@
 $EndComp
 $Comp
-L power:GND #PWR0405
+L power:GND #PWR0303
 U 1 1 5F64278D
 P 5600 3550
-F 0 "#PWR0405" H 5600 3300 50  0001 C CNN
+F 0 "#PWR0303" H 5600 3300 50  0001 C CNN
 F 1 "GND" H 5605 3377 50  0000 C CNN
 F 2 "" H 5600 3550 50  0001 C CNN
@@
 $EndComp
 $Comp
-L power:GND #PWR0402
+L power:GND #PWR0302
 U 1 1 5F642C6B
 P 4500 3250
-F 0 "#PWR0402" H 4500 3000 50  0001 C CNN
+F 0 "#PWR0302" H 4500 3000 50  0001 C CNN
 F 1 "GND" H 4505 3077 50  0000 C CNN
 F 2 "" H 4500 3250 50  0001 C CNN
@@
 $EndComp
 $Comp
-L power:GND #PWR0410
+L power:GND #PWR0304
 U 1 1 5F642EA6
 P 6800 3250
-F 0 "#PWR0410" H 6800 3000 50  0001 C CNN
+F 0 "#PWR0304" H 6800 3000 50  0001 C CNN
 F 1 "GND" H 6805 3077 50  0000 C CNN
 F 2 "" H 6800 3250 50  0001 C CNN
@@
 $EndComp
 $Comp
-L power:+5V #PWR0401
+L power:+5V #PWR0301
 U 1 1 5F643827
 P 4050 2900
-F 0 "#PWR0401" H 4050 2750 50  0001 C CNN
+F 0 "#PWR0301" H 4050 2750 50  0001 C CNN
 F 1 "+5V" H 4065 3073 50  0000 C CNN
 F 2 "" H 4050 2900 50  0001 C CNN
@@
 $EndComp
 $Comp
-L power:+3.3V #PWR0411
+L power:+3.3V #PWR0305
 U 1 1 5F643F44
 P 7050 2800
-F 0 "#PWR0411" H 7050 2650 50  0001 C CNN
+F 0 "#PWR0305" H 7050 2650 50  0001 C CNN
 F 1 "+3.3V" H 7065 2973 50  0000 C CNN
 F 2 "" H 7050 2800 50  0001 C CNN
@@
 	7050 2800 7050 2850
 $Comp
-L power:PWR_FLAG #FLG0110
+L power:PWR_FLAG #FLG0301
 U 1 1 5FD16A71
 P 7050 2850
-F 0 "#FLG0110" H 7050 2925 50  0001 C CNN
+F 0 "#FLG0301" H 7050 2925 50  0001 C CNN
 F 1 "PWR_FLAG" V 7050 2978 50  0000 L CNN
 F 2 "" H 7050 2850 50  0001 C CNN

Commit message: Note: Schmitt trigger for joystick Buttons TODO
Signed-off-by: Eldalote.Electronics <Eldalote.Electronics@gmail.com>
Parts:
- C301, C302: footprint Capacitor_SMD:C_0805_2012Metric_Pad1.15x1.40mm_HandSolder -> Capacitor_SMD:C_0805_2012Metric
Changed lines of the file:
@@
 F 0 "C302" H 6892 3096 50  0000 L CNN
 F 1 "22uF" H 6892 3005 50  0000 L CNN
-F 2 "Capacitor_SMD:C_0805_2012Metric_Pad1.15x1.40mm_HandSolder" H 6800 3050 50  0001 C CNN
+F 2 "Capacitor_SMD:C_0805_2012Metric" H 6800 3050 50  0001 C CNN
 F 3 "~" H 6800 3050 50  0001 C CNN
 F 4 "C45783" H 6800 3050 50  0001 C CNN "LCSC"
@@
 F 0 "C301" H 4592 3096 50  0000 L CNN
 F 1 "10uF" H 4592 3005 50  0000 L CNN
-F 2 "Capacitor_SMD:C_0805_2012Metric_Pad1.15x1.40mm_HandSolder" H 4500 3050 50  0001 C CNN
+F 2 "Capacitor_SMD:C_0805_2012Metric" H 4500 3050 50  0001 C CNN
 F 3 "~" H 4500 3050 50  0001 C CNN
 F 4 "C15850" H 4500 3050 50  0001 C CNN "LCSC"

Commit message: Screen POT->PWM and RGB LEDS reworked, making space on the CPU pins. Almost done
Signed-off-by: Eldalote.Electronics <Eldalote.Electronics@gmail.com>
Parts:
- U301: footprint SOT95P280X145-5N -> SamacSys_Parts:SOT95P280X145-5N
Changed lines of the file:
@@
 F 0 "U301" H 5625 3165 50  0000 C CNN
 F 1 "SC189ZSKTRT" H 5625 3074 50  0000 C CNN
-F 2 "SOT95P280X145-5N" H 6100 3000 50  0001 L CNN
+F 2 "SamacSys_Parts:SOT95P280X145-5N" H 6100 3000 50  0001 L CNN
 F 3 "http://www.semtech.com/images/datasheet/sc189.pdf" H 6100 2900 50  0001 L CNN
 F 4 "Switching Voltage Regulators 2.5MHz-1.5A SYNC STEP DOWN REG" H 6100 2800 50  0001 L CNN "Description"
