File: PCBs/Drone main board/3v3-2v5-regulator.sch (KiCad schematic (older format))
At the start: 7 parts, among them U401 SC189ZSKTRT, U402 NCP115ASN250T2G

Commit message: Lots of work to check every component, add Manufacturers number (instead of LCSC or digikey and mouser numbers)
Changed to USB-C connector, almost done with that sheet. Components checked, need to redo Sheet IO

Signed-off-by: Eldalote.Electronics <Eldalote.Electronics@gmail.com>
Parts:
- C401: LCSC C15850 -> (none); MfNr (none) -> CL21A106KAYNNNG
- C402, C403: LCSC C15849 -> (none); MfNr (none) -> CL10A105KB8NNNC
- C404: LCSC C45783 -> (none); MfNr (none) -> CL21A226MAQNNNE
- L401: DigiKey 445-180921-1-ND -> (none); MfNr (none) -> VLS3012CX-1R0M-1; Mouser 810-VLS3012CX-1R0M-1 -> (none)
- U401: Manufacturer_Name SEMTECH -> (none); Manufacturer_Part_Number SC189ZSKTRT -> (none); MfNr (none) -> SC189ZSKTRT; Mouser Part Number 947-SC189ZSKTRT -> (none); Mouser Price/Stock https://www.mouser.co.uk/ProductDetail/Semtech/SC189ZSKTRT?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 -> (none)
- U402: DigiKey NCP115ASN250T2GOSCT-ND -> (none); MfNr (none) -> NCP115ASN250T2G; Mouser 863-NCP115ASN250T2G -> (none)
Changed lines of the file:
@@
 F 4 "Switching Voltage Regulators 2.5MHz-1.5A SYNC STEP DOWN REG" H 6050 1450 50  0001 L CNN "Description"
 F 5 "1.45" H 6050 1350 50  0001 L CNN "Height"
-F 6 "947-SC189ZSKTRT" H 6050 1250 50  0001 L CNN "Mouser Part Number"
-F 7 "https://www.mouser.co.uk/ProductDetail/Semtech/SC189ZSKTRT?qs=rBWM4%252BvDhIck0D%2FgoUNMIQ%3D%3D" H 6050 1150 50  0001 L CNN "Mouser Price/Stock"
-F 8 "SEMTECH" H 6050 1050 50  0001 L CNN "Manufacturer_Name"
-F 9 "SC189ZSKTRT" H 6050 950 50  0001 L CNN "Manufacturer_Part_Number"
+F 6 "SC189ZSKTRT" H 6050 950 50  0001 L CNN "MfNr"
 	1    5100 1550
 	1    0    0    -1
@@
 F 2 "Capacitor_SMD:C_0805_2012Metric" H 6750 1700 50  0001 C CNN
 F 3 "~" H 6750 1700 50  0001 C CNN
-F 4 "C45783" H 6750 1700 50  0001 C CNN "LCSC"
+F 4 "CL21A226MAQNNNE" H 6750 1700 50  0001 C CNN "MfNr"
 	1    6750 1700
 	1    0    0    -1
@@
 F 2 "Capacitor_SMD:C_0805_2012Metric" H 4450 1700 50  0001 C CNN
 F 3 "~" H 4450 1700 50  0001 C CNN
-F 4 "C15850" H 4450 1700 50  0001 C CNN "LCSC"
+F 4 "CL21A106KAYNNNG" H 4450 1700 50  0001 C CNN "MfNr"
 	1    4450 1700
 	1    0    0    -1
@@
 F 2 "Eldalote-footprints:L_3012_TDK" H 6400 1550 50  0001 C CNN
 F 3 "~" H 6400 1550 50  0001 C CNN
-F 4 "810-VLS3012CX-1R0M-1 " V 6400 1550 50  0001 C CNN "Mouser"
-F 5 "445-180921-1-ND " V 6400 1550 50  0001 C CNN "DigiKey"
+F 4 "VLS3012CX-1R0M-1" V 6400 1550 50  0001 C CNN "MfNr"
 	1    6400 1550
 	0    -1   -1   0
@@
 F 2 "SOT95P275X110-5N" H 6400 4300 50  0001 L CNN
 F 3 "http://www.onsemi.com/pub/Collateral/NCP115-D.PDF" H 6400 4400 50  0001 L CNN
-F 4 "863-NCP115ASN250T2G " H 5150 3850 50  0001 C CNN "Mouser"
-F 5 " NCP115ASN250T2GOSCT-ND " H 5150 3850 50  0001 C CNN "DigiKey"
+F 4 "NCP115ASN250T2G" H 5150 3850 50  0001 C CNN "MfNr"
 	1    5150 3850
 	1    0    0    -1
@@
 F 2 "Capacitor_SMD:C_0603_1608Metric" H 4700 4000 50  0001 C CNN
 F 3 "~" H 4700 4000 50  0001 C CNN
-F 4 "C15849" H 4700 4000 50  0001 C CNN "LCSC"
+F 4 "CL10A105KB8NNNC" H 4700 4000 50  0001 C CNN "MfNr"
 	1    4700 4000
 	1    0    0    -1
@@
 F 2 "Capacitor_SMD:C_0603_1608Metric" H 6400 4000 50  0001 C CNN
 F 3 "~" H 6400 4000 50  0001 C CNN
-F 4 "C15849" H 6400 4000 50  0001 C CNN "LCSC"
+F 4 "CL10A105KB8NNNC" H 6400 4000 50  0001 C CNN "MfNr"
 	1    6400 4000
 	1    0    0    -1
