File: PCBs/Drone main board/Power-Distribution-Estimation.sch (KiCad schematic (older format))
At the start: 2 parts, among them J201 PJ-102A

Commit message: Lots of work to check every component, add Manufacturers number (instead of LCSC or digikey and mouser numbers)
Changed to USB-C connector, almost done with that sheet. Components checked, need to redo Sheet IO

Signed-off-by: Eldalote.Electronics <Eldalote.Electronics@gmail.com>
Parts:
- J201: DigiKey CP-102A-ND -> (none); MfNr (none) -> PJ-102A; Mouser 490-PJ-102A -> (none)
- JP201: DigiKey A860AR-ND -> (none); MfNr (none) -> ME-100; Mouser 535-ME-100 -> (none)
Changed lines of the file:
@@
 F 2 "Connector_PinHeader_2.54mm:PinHeader_1x03_P2.54mm_Vertical" H 8100 5000 50  0001 C CNN
 F 3 "~" H 8100 5000 50  0001 C CNN
-F 4 "535-ME-100 " H 8100 5000 50  0001 C CNN "Mouser"
-F 5 "A860AR-ND" H 8100 5000 50  0001 C CNN "DigiKey"
+F 4 " ME-100 " H 8100 5000 50  0001 C CNN "MfNr"
 	1    8100 5000
 	-1   0    0    1
@@
 F 2 "digikey-footprints:Barrel_Jack_5.5mmODx2.1mmID_PJ-102A" H 7550 5200 60  0001 L CNN
 F 3 "https://www.cui.com/product/resource/digikeypdf/pj-102a.pdf" H 7550 5300 60  0001 L CNN
-F 4 "490-PJ-102A" H 7350 5000 50  0001 C CNN "Mouser"
-F 5 "CP-102A-ND" H 7550 5400 60  0001 L CNN "DigiKey"
+F 4 "PJ-102A" H 7350 5000 50  0001 C CNN "MfNr"
 	1    7350 5000
 	1    0    0    -1
